File: PCB/AURA.kicad_pcb (KiCad board)
At the start: 2 copper layers, 69 x 43.3 mm, 60 parts, among them J1 USB_C_Receptacle_USB2.0_16P, J11 Conn_01x03_Pin, J12 Conn_01x03_Pin, J13 Conn_01x04_Pin, J2 Conn_01x02_Pin, J3 Conn_01x03_Pin, J4 Conn_01x02_Pin, J5 Conn_01x03_Pin, J6 Conn_01x02_Pin, Q1 AO3401A, SW1 SW_DPDT_x2, SW2 SW_Push, U1 AP63203WU, U2 L7805, U3 MPU-6050, U4 BMP280, U5 ICM-20948, U6 LD39015M18R, U7 STM32F401CBUx, Y1 Crystal_GND24_Small

Commit message: Add files via upload
Parts:
- removed C1: 2u2, Capacitor_SMD:C_0201_0603Metric
- removed R5: 100R, Resistor_SMD:R_0603_1608Metric
- added D4: 1N4001, Diode_THT:D_DO-41_SOD81_P5.08mm_Vertical_AnodeUp, F.Cu at (151.0, 77.2)
- added L1: 2.2uh, Inductor_SMD:L_0603_1608Metric, F.Cu at (147.5, 80.5)
- added L2: 4.7uf, Inductor_SMD:L_0603_1608Metric, F.Cu at (154.5, 77.0)
- C2: value 2u2 -> 47uf
- C3: value 2u2 -> 10uf
- C6: value 100n -> 22uf
- moved C3 1.08 mm to (151.0, 80.9)
- moved C2 1.05 mm to (152.0, 81.0)
Connections:
- C18 pad 2: Net-(U6-GND) -> GND
- C19 pad 2: Net-(U6-GND) -> GND
- U1 pad 1: 3.3V -> Net-(U1-FB)
- U6 pad 2: Net-(U6-GND) -> GND
- U6 pad 3: unconnected-(U6-EN-Pad3) -> 3.3V
Routing:
- net GND: track 111.9 -> 129.7 mm, vias 14 -> 16
- net Net-(U6-GND): track 5.45 -> 0.00 mm
- net 3.3V: track 123.9 -> 128.1 mm
- net Net-(D4-K): track 6.42 -> 10.4 mm
- net Net-(U1-FB): track 0.00 -> 1.80 mm
- added copper zone on F.Cu, net (none)
