File: PCB/AURA.kicad_sch (KiCad schematic)
At the start: 60 parts, among them J1 USB_C_Receptacle_USB2.0_16P, J11 Conn_01x03_Pin, J12 Conn_01x03_Pin, J13 Conn_01x04_Pin, J2 Conn_01x02_Pin, J3 Conn_01x03_Pin, J4 Conn_01x02_Pin, J5 Conn_01x03_Pin, J6 Conn_01x02_Pin, Q1 AO3401A, SW1 SW_DPDT_x2, SW2 SW_Push, U1 AP63203WU, U2 L7805, U3 MPU-6050, U4 BMP280, U5 ICM-20948, U6 LD39015M18R, U7 STM32F401CBUx, Y1 Crystal_GND24_Small

Commit message: Add files via upload
Parts:
- removed C1: 2u2, Capacitor_SMD:C_0201_0603Metric, symbol Device:C
- removed R5: 100R, Resistor_SMD:R_0603_1608Metric, symbol Device:R
- added D4: 1N4001, Diode_THT:D_DO-41_SOD81_P5.08mm_Vertical_AnodeUp, symbol Diode:1N4001
- added L1: 2.2uh, Inductor_SMD:L_0603_1608Metric, symbol Device:L
- added L2: 4.7uf, Inductor_SMD:L_0603_1608Metric, symbol Device:L
- C2: value 2u2 -> 47uf
- C3: value 2u2 -> 10uf
- C6: value 100n -> 22uf
Connections:
- net 3.3V: now also U6.3 (EN), L2.2; no longer U1.1 (FB)
- net GND: now also C18.2, C19.2, U6.2 (GND), D4.2 (A)
- net at F1.2: now also L1.1
- net at C2.1, C3.1, U1.2 (EN)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: now also D4.1 (K), L1.2
- new net: L2.1, U1.1 (FB)
