File: PCB/ESC/AURA_ESC.kicad_pcb (KiCad board)
At the start: 4 copper layers, 61.9 x 37.7 mm, 70 parts, among them J1 Conn_01x03_Pin, J2 Conn_01x04_Pin, J3 Conn_01x01_Pin, J4 Conn_01x01_Pin, J5 Conn_01x01_Pin, J6 Conn_01x01_Pin, J7 Conn_01x01_Pin, U1 STM32F051K8U6, U10 SQJ138ELP-T1_GE3, U2 INA199A1DCKR, U3 AOZ1282CI, U4 AMS1117-3.3, U5 SQJ138ELP-T1_GE3, U6 SQJ138ELP-T1_GE3, U7 SQJ138ELP-T1_GE3, U8 SQJ138ELP-T1_GE3, U9 SQJ138ELP-T1_GE3

Commit message: Add files via upload
Parts:
- removed U4: AMS1117-3.3, Package_TO_SOT_SMD:SOT-223-3_TabPin2
- added C19: 22uf, Capacitor_SMD:C_0201_0603Metric, F.Cu at (139.5, 86.8)
- added C20: 47uf, Capacitor_SMD:C_0201_0603Metric, F.Cu at (128.3, 86.8)
- added C21: 100n, Capacitor_SMD:C_0201_0603Metric, F.Cu at (136.0, 87.2)
- added U12: AP63203WU, Package_TO_SOT_SMD:TSOT-23-6, F.Cu at (133.4, 87.4)
- moved C5 0.91 mm to (129.9, 88.1)
- moved C4 0.90 mm to (137.8, 88.1), turned to -90 degrees
Routing:
- net Vcc_M: track 217.6 -> 239.7 mm, vias 13 -> 10
- net gnd_p: track 391.4 -> 406.3 mm, vias 12 -> 13
- net VDD: track 127.3 -> 120.0 mm, vias 5 -> 6
- net Vcc: track 48.4 -> 43.3 mm
- net /+10v: track 78.9 -> 82.9 mm
- net (no net): track 0.00 -> 2.54 mm, vias 18 -> 16
